Commit message: Add flipped inflated gripper URDF

File: urdf/wsg50_flipped_inflated.urdf (robot description, URDF)
Before this commit: robot float_wsg50, 13 links, 12 joints
Links:
- link wsg50_finger_left: geometry collision mesh filename=package://meshes/bubbles/collision/bubble_flipped_inflated.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 scale=0.001 0.001 0.001; visual mesh filename=package://meshes/bubbles/collision/bubble_flipped_inflated.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 scale=0.001 0.001 0.001
- link wsg50_finger_right: geometry collision mesh filename=package://meshes/bubbles/visual/bubble_flipped_inflated.stl scale=0.001 0.001 0.001; visual mesh filename=package://meshes/bubbles/collision/bubble_flipped_inflated.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 scale=0.001 0.001 0.001
Joints:
- joint wsg50_grasp_frame_fake_joint: origin xyz=0 0 0.194 rpy=0 0 0 -> (none)
