Commit message: Add drill and hammer objects for experiments

File: urdf/YcbHammer/model.urdf (robot description, URDF)
Before this commit: robot model.urdf, 1 links, 0 joints
Links:
- link baseLink: geometry collision mesh filename=collision_vhacd.obj scale=1 1 1; visual mesh filename=textured_simple_reoriented.obj scale=1 1 1
