Commit message: Add spam can poke experiments

File: urdf/YcbMasterChefCan/model.urdf (robot description, URDF)
Before this commit: robot model.urdf, 1 links, 0 joints
Links:
- link baseLink: geometry collision mesh filename=collision_vhacd.obj scale=1.0 1.0 1.0; visual mesh filename=textured_simple_reoriented.obj scale=1.0 1.0 1.0
